Commit message: Sync end-tool offset changes from server kinematics.urdf to electron-app
Reduce tool_vacuum and tool_servo z-offsets to match the updated server-side URDF.

File: electron-app/kinematics.urdf (robot description, URDF)
Before this commit: robot matrix_arm_v3, 12 links, 11 joints
Joints:
- joint tool_servo: origin xyz=0 0 -0.15219 rpy=0 0 0 -> xyz=0 0 -0.12019 rpy=0 0 0
- joint tool_vacuum: origin xyz=0 0 -0.14062 rpy=0 0 0 -> xyz=0 0 -0.10862 rpy=0 0 0
