Commit message: Limit all 6 joints to +/-90 degrees in URDF
Tightens joint limits from their previous values (some were +/-180 or +/-100 degrees)
to +/-1.5708 rad (+/-90 deg) on all joints. This prevents IK from finding solutions
that require joints to pass through or near singularities and avoids the observed
180-degree wrist inversion.

Co-Authored-By: Claude Sonnet 4.6 <noreply@anthropic.com>

File: electron-app/kinematics.urdf (robot description, URDF)
Before this commit: robot matrix_arm_v3, 8 links, 7 joints
Joints:
- joint joint1_base_yaw: limit lower=-3.14 upper=3.14 effort=10 velocity=2 -> lower=-1.5708 upper=1.5708 effort=10 velocity=2
- joint joint2_shoulder_pitch: limit lower=-1.57 upper=1.57 effort=10 velocity=2 -> lower=-1.5708 upper=1.5708 effort=10 velocity=2
- joint joint3_elbow_pitch: limit lower=-1.74533 upper=1.74533 effort=10 velocity=2 -> lower=-1.5708 upper=1.5708 effort=10 velocity=2
- joint joint4_wrist_roll: limit lower=-3.14 upper=3.14 effort=5 velocity=3 -> lower=-1.5708 upper=1.5708 effort=5 velocity=3
- joint joint5_wrist_pitch: limit lower=-1.57 upper=1.57 effort=5 velocity=3 -> lower=-1.5708 upper=1.5708 effort=5 velocity=3
- joint joint6_wrist_roll_2: limit lower=-3.14 upper=3.14 effort=5 velocity=3 -> lower=-1.5708 upper=1.5708 effort=5 velocity=3

Commit message: Restore J1 base yaw to +/-180 degrees
Co-Authored-By: Claude Sonnet 4.6 <noreply@anthropic.com>

File: electron-app/kinematics.urdf (robot description, URDF)
Before this commit: robot matrix_arm_v3, 8 links, 7 joints
Joints:
- joint joint1_base_yaw: limit lower=-1.5708 upper=1.5708 effort=10 velocity=2 -> lower=-3.14159 upper=3.14159 effort=10 velocity=2

Commit message: Flip J2 and J5 axis directions in URDF — physical servos rotate opposite to model
J2 (shoulder pitch) and J5 (wrist pitch) were rotating backwards: positive
commanded angles moved the physical joint in the negative direction. Changing
both from axis xyz="0 1 0" to xyz="0 -1 0" corrects the sign so the IK
output matches physical motion.

J3 already had axis xyz="0 -1 0" so is unchanged.

Co-Authored-By: Claude Sonnet 4.6 <noreply@anthropic.com>

File: electron-app/kinematics.urdf (robot description, URDF)
Before this commit: robot matrix_arm_v3, 8 links, 7 joints
Joints:
- joint joint2_shoulder_pitch: axis 0 1 0 -> 0 -1 0
- joint joint5_wrist_pitch: axis 0 1 0 -> 0 -1 0

Commit message: Update kinematics for electron app and Node.js server
Co-Authored-By: Claude Sonnet 4.6 <noreply@anthropic.com>

File: electron-app/kinematics.urdf (robot description, URDF)
Before this commit: robot matrix_arm_v3, 8 links, 7 joints
Joints:
- joint joint2_shoulder_pitch: limit lower=-1.5708 upper=1.5708 effort=10 velocity=2 -> lower=-1.5708 upper=0.698132 effort=10 velocity=2
- joint joint5_wrist_pitch: limit lower=-1.5708 upper=1.5708 effort=5 velocity=3 -> lower=-0.0872665 upper=1.5708 effort=5 velocity=3

Commit message: Add end-tool auto-detection/kinematics sync, fix OSK script tag dropped in touch-mode pass
- Adds a kinematics tab panel showing the detected end tool and its
  offset table, backed by a Pi-side kinematicsService/server change and
  a REGISTER_MAP update for tool auto-detection.
- Adds sync-urdf.js to regenerate the Pi's kinematics.urdf copy and the
  DEFAULT_URDF fallback embedded in app.js from the single source file,
  wired into postinstall via package.json.
- Restores the <script src="keyboard.js"> tag in index.html, which was
  accidentally dropped in the touch-mode UX pass commit (8693505) —
  this is what stopped the on-screen keyboard from appearing.

Co-Authored-By: Claude Sonnet 5 <noreply@anthropic.com>

File: electron-app/kinematics.urdf (robot description, URDF)
Before this commit: robot matrix_arm_v3, 8 links, 7 joints
Links:
- added link tcp_pen
- added link tcp_servo
- added link tcp_unassigned
- added link tcp_vacuum
Joints:
- added joint tool_pen: type fixed, parent tool_link, child tcp_pen, origin xyz=0 0 -0.155 rpy=0 0 0
- added joint tool_servo: type fixed, parent tool_link, child tcp_servo, origin xyz=0 0 -0.15219 rpy=0 0 0
- added joint tool_unassigned: type fixed, parent tool_link, child tcp_unassigned, origin xyz=0 0 0 rpy=0 0 0
- added joint tool_vacuum: type fixed, parent tool_link, child tcp_vacuum, origin xyz=0 0 -0.14062 rpy=0 0 0

Commit message: Update kinematics.urdf link offsets
Co-Authored-By: Claude Sonnet 5 <noreply@anthropic.com>

File: electron-app/kinematics.urdf (robot description, URDF)
Before this commit: robot matrix_arm_v3, 12 links, 11 joints
Joints:
- joint joint1_base_yaw: origin xyz=0 0 0.05 rpy=0 0 0 -> xyz=0 0 0.03538 rpy=0 0 0
- joint joint2_shoulder_pitch: origin xyz=0 0 0.058 rpy=0 0 0 -> xyz=0 0 0.08553 rpy=0 0 0
- joint joint3_elbow_pitch: origin xyz=0 0 0.135 rpy=0 0 0 -> xyz=0 0 0.11342 rpy=0 0 0
- joint joint4_wrist_roll: origin xyz=0.03965 0 0.055 rpy=0 0 0 -> xyz=0.02498 0 0.055 rpy=0 0 0
- joint joint5_wrist_pitch: origin xyz=0.06285 0 0 rpy=0 0 0 -> xyz=0.08148 0 0 rpy=0 0 0
- joint joint6_wrist_roll_2: origin xyz=0.055 0 -0.03965 rpy=0 0 0 -> xyz=0.055 0 -0.02498 rpy=0 0 0
- joint tool_mount: origin xyz=0 0 -0.035 rpy=0 0 0 -> xyz=0 0 -0.04463 rpy=0 0 0
- joint tool_vacuum: origin xyz=0 0 -0.10862 rpy=0 0 0 -> xyz=0.00202 0 -0.11462 rpy=0 0 0

Commit message: Update kinematics.urdf link offsets
Co-Authored-By: Claude Sonnet 5 <noreply@anthropic.com>

File: electron-app/kinematics.urdf (robot description, URDF)
Before this commit: robot matrix_arm_v3, 12 links, 11 joints
Joints:
- joint joint1_base_yaw: origin xyz=0 0 0.03538 rpy=0 0 0 -> xyz=0 0 0.036 rpy=0 0 0
- joint joint2_shoulder_pitch: origin xyz=0 0 0.08553 rpy=0 0 0 -> xyz=0 0 0.086 rpy=0 0 0

Commit message: Update kinematics.urdf link offsets
Co-Authored-By: Claude Sonnet 5 <noreply@anthropic.com>

File: electron-app/kinematics.urdf (robot description, URDF)
Before this commit: robot matrix_arm_v3, 12 links, 11 joints
Joints:
- joint joint3_elbow_pitch: origin xyz=0 0 0.11342 rpy=0 0 0 -> xyz=0 0 0.113 rpy=0 0 0
- joint tool_mount: origin xyz=0 0 -0.04463 rpy=0 0 0 -> xyz=0 0 -0.05 rpy=0 0 0

Commit message: Update kinematics.urdf link offsets
Co-Authored-By: Claude Sonnet 5 <noreply@anthropic.com>

File: electron-app/kinematics.urdf (robot description, URDF)
Before this commit: robot matrix_arm_v3, 12 links, 11 joints
Joints:
- joint tool_vacuum: origin xyz=0.00202 0 -0.11462 rpy=0 0 0 -> xyz=0.00202 0 -0.119 rpy=0 0 0

Commit message: Update kinematics.urdf in app and server
Co-Authored-By: Claude Sonnet 5 <noreply@anthropic.com>

File: electron-app/kinematics.urdf (robot description, URDF)
Before this commit: robot matrix_arm_v3, 12 links, 11 joints
Joints:
- joint joint6_wrist_roll_2: axis 1 0 0 -> 0 0 1

Commit message: URDF: joint 1 and joint 4 axes flipped to match the real servos (right-handed frame)
Verified on the arm: joint 1 positive turns clockwise from above and
joint 4 positive rolls anticlockwise viewed from behind, both opposite to
the modelled axes. With joint 1 mirrored, every Cartesian Y was reversed
relative to the model and the joint 6 spin compensation ran the wrong way
as the base swung (tool visibly rotated instead of staying world-aligned).
Joint 1 axis is now (0 0 -1) and joint 4 (-1 0 0) in both URDF copies and
the DEFAULT_URDF fallback; joint 6 (verified anticlockwise from above) is
unchanged. The frame is now right-handed: +X forward, +Y on the
anticlockwise side, +Z up. Stored XYZ positions, dead zones and marker
layouts entered under the old convention need their Y sign flipped.

Co-Authored-By: Claude Fable 5.1 <noreply@anthropic.com>

File: electron-app/kinematics.urdf (robot description, URDF)
Before this commit: robot matrix_arm_v3, 12 links, 11 joints
Joints:
- joint joint1_base_yaw: axis 0 0 1 -> 0 0 -1
- joint joint4_wrist_roll: axis 1 0 0 -> -1 0 0

Commit message: URDF: servo gripper TCP is 130 mm below the mount face (measured), not 120.19
Measured on the arm with a rule from the mount face to the closed finger
tips. The model was 10 mm optimistic about tip height with this tool.

Co-Authored-By: Claude Fable 5.1 <noreply@anthropic.com>

File: electron-app/kinematics.urdf (robot description, URDF)
Before this commit: robot matrix_arm_v3, 12 links, 11 joints
Joints:
- joint tool_servo: origin xyz=0 0 -0.12019 rpy=0 0 0 -> xyz=0 0 -0.130 rpy=0 0 0
